File: main_board/EENLD_main/ASP.kicad_sch (KiCad schematic)
At the start: 26 parts, among them U701 74HC4052, U702 TLV9002, U703 TLV9002

Commit message: Finished PCB layout v0.1.
Parts:
- C701, C702, C703: footprint (none) -> Capacitor_SMD:C_0603_1608Metric_Pad1.08x0.95mm_HandSolder; LCSC (none) -> C14663
- R701, R702, R705, R706, R709, R710, R713, R714: footprint (none) -> Resistor_SMD:R_0402_1005Metric_Pad0.72x0.64mm_HandSolder; LCSC (none) -> C25744
- R703, R704, R707, R708, R711, R712, R715, R716: footprint (none) -> Resistor_SMD:R_0402_1005Metric_Pad0.72x0.64mm_HandSolder; LCSC (none) -> C25764
- TP701, TP702, TP703, TP704: footprint (none) -> TestPoint:TestPoint_THTPad_D1.5mm_Drill0.7mm
- U701: footprint Package_SO:SO-16_3.9x9.9mm_P1.27mm -> Package_SO:TSSOP-16_4.4x5mm_P0.65mm; LCSC (none) -> C5646
- U702, U703: footprint Package_SO:SOIC-8_3.9x4.9mm_P1.27mm -> Package_SO:TSSOP-8_4.4x3mm_P0.65mm; LCSC (none) -> C398360

Commit message: added midi2array
Parts:
- TP701, TP702, TP703, TP704: now left out of the parts list
- U701: JLCPCB Rotation Offset (none) -> -90
- U702, U703: JLCPCB Rotation Offset (none) -> -90; LCSC C398360 -> C398359
Changed lines of the file:
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@@
   )
   (symbol (lib_id "Connector:TestPoint") (at 34.3245 146.6159 270) (unit 1)
-    (in_bom yes) (on_board yes) (dnp no) (fields_autoplaced)
+    (in_bom no) (on_board yes) (dnp no) (fields_autoplaced)
     (property "Reference" "TP704" (at 39.4045 145.3459 90)
       (effects (font (size 1.27 1.27)) (justify left))
@@
       (effects (font (size 1.27 1.27)) hide)
     )
-    (property "JLCPCB Rotation Offset" "" (at 50.8 69.85 0)
+    (property "JLCPCB Rotation Offset" "-90" (at 50.8 69.85 0)
       (effects (font (size 1.27 1.27)) hide)
     )
@@
       (effects (font (size 1.27 1.27)) hide)
     )
-    (property "JLCPCB Rotation Offset" "" (at 251.46 87.63 0)
-      (effects (font (size 1.27 1.27)) hide)
-    )
-    (property "LCSC" "C398360" (at 251.46 87.63 0)
+    (property "JLCPCB Rotation Offset" "-90" (at 251.46 87.63 0)
+      (effects (font (size 1.27 1.27)) hide)
+    )
+    (property "LCSC" "C398359" (at 251.46 87.63 0)
       (effects (font (size 1.27 1.27)) hide)
     )
@@
       (effects (font (size 1.27 1.27)) hide)
     )
-    (property "JLCPCB Rotation Offset" "" (at 251.46 48.26 0)
-      (effects (font (size 1.27 1.27)) hide)
-    )
-    (property "LCSC" "C398360" (at 251.46 48.26 0)
+    (property "JLCPCB Rotation Offset" "-90" (at 251.46 48.26 0)
+      (effects (font (size 1.27 1.27)) hide)
+    )
+    (property "LCSC" "C398359" (at 251.46 48.26 0)
       (effects (font (size 1.27 1.27)) hide)
     )
@@
       (effects (font (size 1.27 1.27)) hide)
     )
-    (property "JLCPCB Rotation Offset" "" (at 214.63 93.98 0)
-      (effects (font (size 1.27 1.27)) hide)
-    )
-    (property "LCSC" "C398360" (at 214.63 93.98 0)
+    (property "JLCPCB Rotation Offset" "-90" (at 214.63 93.98 0)
+      (effects (font (size 1.27 1.27)) hide)
+    )
+    (property "LCSC" "C398359" (at 214.63 93.98 0)
       (effects (font (size 1.27 1.27)) hide)
     )
@@
   )
   (symbol (lib_id "Connector:TestPoint") (at 34.29 139.7 270) (unit 1)
-    (in_bom yes) (on_board yes) (dnp no) (fields_autoplaced)
+    (in_bom no) (on_board yes) (dnp no) (fields_autoplaced)
     (property "Reference" "TP703" (at 39.37 138.43 90)
       (effects (font (size 1.27 1.27)) (justify left))
@@
   )
   (symbol (lib_id "Connector:TestPoint") (at 34.29 133.35 270) (unit 1)
-    (in_bom yes) (on_board yes) (dnp no) (fields_autoplaced)
+    (in_bom no) (on_board yes) (dnp no) (fields_autoplaced)
     (property "Reference" "TP702" (at 39.37 132.08 90)
       (effects (font (size 1.27 1.27)) (justify left))
@@
       (effects (font (size 1.27 1.27)) hide)
     )
-    (property "JLCPCB Rotation Offset" "" (at 157.48 87.63 0)
-      (effects (font (size 1.27 1.27)) hide)
-    )
-    (property "LCSC" "C398360" (at 157.48 87.63 0)
+    (property "JLCPCB Rotation Offset" "-90" (at 157.48 87.63 0)
+      (effects (font (size 1.27 1.27)) hide)
+    )
+    (property "LCSC" "C398359" (at 157.48 87.63 0)
       (effects (font (size 1.27 1.27)) hide)
     )
@@
       (effects (font (size 1.27 1.27)) hide)
     )
-    (property "JLCPCB Rotation Offset" "" (at 157.48 48.26 0)
-      (effects (font (size 1.27 1.27)) hide)
-    )
-    (property "LCSC" "C398360" (at 157.48 48.26 0)
+    (property "JLCPCB Rotation Offset" "-90" (at 157.48 48.26 0)
+      (effects (font (size 1.27 1.27)) hide)
+    )
+    (property "LCSC" "C398359" (at 157.48 48.26 0)
       (effects (font (size 1.27 1.27)) hide)
     )
@@
       (effects (font (size 1.27 1.27)) hide)
     )
-    (property "JLCPCB Rotation Offset" "" (at 120.65 93.98 0)
-      (effects (font (size 1.27 1.27)) hide)
-    )
-    (property "LCSC" "C398360" (at 120.65 93.98 0)
+    (property "JLCPCB Rotation Offset" "-90" (at 120.65 93.98 0)
+      (effects (font (size 1.27 1.27)) hide)
+    )
+    (property "LCSC" "C398359" (at 120.65 93.98 0)
       (effects (font (size 1.27 1.27)) hide)
     )
@@
   )
   (symbol (lib_id "Connector:TestPoint") (at 34.29 127 270) (unit 1)
-    (in_bom yes) (on_board yes) (dnp no) (fields_autoplaced)
+    (in_bom no) (on_board yes) (dnp no) (fields_autoplaced)
     (property "Reference" "TP701" (at 39.37 125.73 90)
       (effects (font (size 1.27 1.27)) (justify left))
